File: Odometre/Hardware/Odometre_Schematic/_autosave-Odometre_Schematic.kicad_sch (KiCad schematic)
At the start: 7 parts, among them J1 Conn_01x04_Pin, J2 Conn_01x08_Pin, U1 MCP2562-E-SN

Commit message: schematic kicad
Parts:
- added U2: LM1117DT-3.3, Package_TO_SOT_SMD:TO-252-3_TabPin2, symbol Regulator_Linear:LM1117DT-3.3
Changed lines of the file:
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@@
+    )
+  )
+  (symbol (lib_id "Regulator_Linear:LM1117DT-3.3") (at 162.56 48.26 0) (unit 1)
+    (in_bom yes) (on_board yes) (dnp no) (fields_autoplaced)
+    (property "Reference" "U2" (at 162.56 41.91 0)
+      (effects (font (size 1.27 1.27)))
+    )
+    (property "Value" "LM1117DT-3.3" (at 162.56 44.45 0)
+      (effects (font (size 1.27 1.27)))
+    )
+    (property "Footprint" "Package_TO_SOT_SMD:TO-252-3_TabPin2" (at 162.56 48.26 0)
+      (effects (font (size 1.27 1.27)) hide)
+    )
+    (property "Datasheet" "http://www.ti.com/lit/ds/symlink/lm1117.pdf" (at 162.56 48.26 0)
+      (effects (font (size 1.27 1.27)) hide)
+    )
+    (pin "1")
+    (pin "2")
+    (pin "3")
+    (instances
+      (project "Odometre_Schematic"
+        (path "/3741a7b9-879e-49a1-88bd-82d63456a983"
+          (reference "U2") (unit 1)
+        )
+      )
     )
   )
