File: Odometre/Hardware/Odometre_Schematic/Odometre_Schematic.kicad_pcb (KiCad board)
At the start: 2 copper layers, 35 parts, among them IC1 STM32C092FCP6, J1 Conn_01x03_Pin, J2 Conn_01x03_Pin, J3 Conn_Alim, J4 Conn_Laser1, J5 Conn_Laser2, J6 Conn_01x06_Pin, J7 Conn_01x06_Pin, SW1 Reset_Botton, SW2 Debug_Botton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

Commit message: shematic+pcb
Parts:
- moved H2 60.4 mm to (188.5, 65.0)
- moved H4 57.0 mm to (189.0, 115.0)
- moved R4 50.5 mm to (122.1, 73.0)
- moved D3 46.9 mm to (122.1, 77.0)
- moved J3 37.0 mm to (123.6, 105.6), turned to 180 degrees
- moved D2 35.3 mm to (154.6, 73.2)
- moved C6 35.3 mm to (139.5, 59.8)
- moved R2 35.3 mm to (166.8, 56.7)
- moved R3 35.3 mm to (166.8, 59.2)
- moved SW1 35.3 mm to (143.9, 54.9)
- moved SW2 35.3 mm to (143.9, 63.5)
- moved D1 35.3 mm to (154.6, 70.6)
- moved J1 35.3 mm to (144.2, 45.5)
- moved J2 35.3 mm to (148.8, 45.5)
- moved J6 35.3 mm to (153.3, 45.5)
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Routing:
- added copper zone on B.Cu, net (none)
- added copper zone on F.Cu, net (none)
Other:
- board outline added: 83.2 x 61.6 mm

Commit message: modifs che pas
Parts:
- removed SW1: Reset_Botton, Button_Switch_THT:SW_PUSH_6mm
- removed SW2: Debug_Botton, Button_Switch_THT:SW_PUSH_6mm
- added S1: 430182043816, projo:430182043816, F.Cu at (175.0, 63.4)
- added S2: 430182043816, projo:430182043816, F.Cu at (175.0, 71.2)
- J1, J2: footprint Connector_PinHeader_2.54mm:PinHeader_1x03_P2.54mm_Vertical -> Connector_JST:JST_PH_B3B-PH-K_1x03_P2.00mm_Vertical
- J4, J5: footprint Connector_PinSocket_2.54mm:PinSocket_1x02_P2.54mm_Vertical -> Connector_PinHeader_2.54mm:PinHeader_1x03_P2.54mm_Vertical
- J6: footprint Connector_PinHeader_2.54mm:PinHeader_1x03_P2.54mm_Vertical -> Connector_PinHeader_2.54mm:PinHeader_1x06_P2.54mm_Vertical
- J7: footprint Connector_PinHeader_2.54mm:PinHeader_1x03_P2.54mm_Vertical -> Connector_JST:JST_PH_B6B-PH-K_1x06_P2.00mm_Vertical
Connections:
- C1 pad 1: ALIM_Trans -> Alim
- C8 pad 1: ALIM_Trans -> Alim
- J3 pad 1: ALIM_Trans -> Alim
- U2 pad 3: ALIM_Trans -> Alim
- U3 pad 3: ALIM_Trans -> Alim
