File: Datalogger/Hardware/Datalogger.kicad_sch (KiCad schematic)
At the start: 27 parts, among them J1 SD_Card, J2 Conn_01x03_Pin, J3 Conn_01x03_Pin, J4 Conn_01x06_Pin, J5 Conn_01x04_Pin, J6 Conn_01x02_Pin, SW1 SW_Push, SW2 SW_SPST, U1 STM32F042F6Px, U2 LM1117DT-3.3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

Commit message: read me datalogger
Parts:
- C1, C2, C3: footprint (none) -> Capacitor_SMD:C_0603_1608Metric_Pad1.08x0.95mm_HandSolder
- D1, D2, D3: footprint (none) -> Diode_SMD:D_0603_1608Metric_Pad1.05x0.95mm_HandSolder
- H1, H2, H3, H4: footprint (none) -> MountingHole:MountingHole_3.2mm_M3_DIN965_Pad
- J1: footprint (none) -> Connector_Card:microSD_HC_Molex_104031-0811
- J2, J3: footprint (none) -> Connector:FanPinHeader_1x03_P2.54mm_Vertical
- J4: footprint (none) -> Connector_PinHeader_2.54mm:PinHeader_1x06_P2.54mm_Vertical
- J5: footprint (none) -> Connector:FanPinHeader_1x04_P2.54mm_Vertical
- J6: footprint (none) -> Connector_JST:JST_XH_B2B-XH-A_1x02_P2.50mm_Vertical
- R1, R2, R3, R4, R5, R6: footprint (none) -> Resistor_SMD:R_0603_1608Metric_Pad0.98x0.95mm_HandSolder
- SW1, SW2: footprint (none) -> Button_Switch_SMD:SW_SPST_EVQPE1
