File: Datalogger/Hardware/Datalogger.kicad_sch (KiCad schematic)
At the start: 22 parts, among them J1 SD_Card, J2 Conn_01x03_Pin, J3 Conn_01x03_Pin, SW1 SW_Push, SW2 SW_SPST, U1 STM32F042F6Px, U2 LM1117DT-3.3, U3 MCP2562-E-SN

Commit message: Modif affectation
Parts:
- C1, C2: footprint (none) -> Capacitor_SMD:C_0805_2012Metric_Pad1.18x1.45mm_HandSolder
- C3: renamed from C; footprint (none) -> Capacitor_SMD:C_0805_2012Metric_Pad1.18x1.45mm_HandSolder
- D1, D2: footprint (none) -> Diode_SMD:D_0201_0603Metric_Pad0.64x0.40mm_HandSolder
- H1, H2, H3, H4: footprint (none) -> MountingHole:MountingHole_2.2mm_M2_DIN965_Pad
- R1, R2, R3, R4, R5: footprint (none) -> Resistor_SMD:R_0603_1608Metric_Pad0.98x0.95mm_HandSolder
Changed lines of the file:
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@@
       (effects (font (size 1.27 1.27)))
     )
-    (property "Footprint" "" (at 45.72 131.572 90)
+    (property "Footprint" "Resistor_SMD:R_0603_1608Metric_Pad0.98x0.95mm_HandSolder" (at 45.72 131.572 90)
       (effects (font (size 1.27 1.27)) hide)
     )
@@
       (effects (font (size 1.27 1.27)) (justify left))
     )
-    (property "Footprint" "" (at 149.86 110.49 0)
+    (property "Footprint" "MountingHole:MountingHole_2.2mm_M2_DIN965_Pad" (at 149.86 110.49 0)
       (effects (font (size 1.27 1.27)) hide)
     )
@@
       (effects (font (size 1.27 1.27)))
     )
-    (property "Footprint" "" (at 161.29 50.8 0)
+    (property "Footprint" "Diode_SMD:D_0201_0603Metric_Pad0.64x0.40mm_HandSolder" (at 161.29 50.8 0)
       (effects (font (size 1.27 1.27)) hide)
     )
@@
   (symbol (lib_id "Device:C") (at 46.99 43.18 180) (unit 1)
     (in_bom yes) (on_board yes) (dnp no)
-    (property "Reference" "C" (at 41.91 40.64 0)
+    (property "Reference" "C3" (at 41.91 40.64 0)
       (effects (font (size 1.27 1.27)) (justify right))
     )
@@
       (effects (font (size 1.27 1.27)) (justify right))
     )
-    (property "Footprint" "" (at 46.0248 39.37 0)
+    (property "Footprint" "Capacitor_SMD:C_0805_2012Metric_Pad1.18x1.45mm_HandSolder" (at 46.0248 39.37 0)
       (effects (font (size 1.27 1.27)) hide)
     )
@@
       (project "Datalogger"
         (path "/4491823b-09d4-418b-ab54-8475663bcb45"
-          (reference "C") (unit 1)
+          (reference "C3") (unit 1)
         )
       )
@@
       (effects (font (size 1.27 1.27)))
     )
-    (property "Footprint" "" (at 153.67 35.052 90)
+    (property "Footprint" "Resistor_SMD:R_0603_1608Metric_Pad0.98x0.95mm_HandSolder" (at 153.67 35.052 90)
       (effects (font (size 1.27 1.27)) hide)
     )
@@
       (effects (font (size 1.27 1.27)))
     )
-    (property "Footprint" "" (at 45.72 136.652 90)
+    (property "Footprint" "Resistor_SMD:R_0603_1608Metric_Pad0.98x0.95mm_HandSolder" (at 45.72 136.652 90)
       (effects (font (size 1.27 1.27)) hide)
     )
@@
       (effects (font (size 1.27 1.27)) (justify left))
     )
-    (property "Footprint" "" (at 149.86 128.27 0)
+    (property "Footprint" "MountingHole:MountingHole_2.2mm_M2_DIN965_Pad" (at 149.86 128.27 0)
       (effects (font (size 1.27 1.27)) hide)
     )
@@
       (effects (font (size 1.27 1.27)) (justify left))
     )
-    (property "Footprint" "" (at 149.86 119.38 0)
+    (property "Footprint" "MountingHole:MountingHole_2.2mm_M2_DIN965_Pad" (at 149.86 119.38 0)
       (effects (font (size 1.27 1.27)) hide)
     )
@@
       (effects (font (size 1.27 1.27)) (justify left))
     )
-    (property "Footprint" "" (at 254.9652 133.35 0)
+    (property "Footprint" "Capacitor_SMD:C_0805_2012Metric_Pad1.18x1.45mm_HandSolder" (at 254.9652 133.35 0)
       (effects (font (size 1.27 1.27)) hide)
     )
@@
       (effects (font (size 1.27 1.27)))
     )
-    (property "Footprint" "" (at 45.72 123.952 90)
+    (property "Footprint" "Resistor_SMD:R_0603_1608Metric_Pad0.98x0.95mm_HandSolder" (at 45.72 123.952 90)
       (effects (font (size 1.27 1.27)) hide)
     )
@@
       (effects (font (size 1.27 1.27)) (justify left))
     )
-    (property "Footprint" "" (at 209.2452 133.35 0)
+    (property "Footprint" "Capacitor_SMD:C_0805_2012Metric_Pad1.18x1.45mm_HandSolder" (at 209.2452 133.35 0)
       (effects (font (size 1.27 1.27)) hide)
     )
@@
       (effects (font (size 1.27 1.27)))
     )
-    (property "Footprint" "" (at 153.67 49.022 90)
+    (property "Footprint" "Resistor_SMD:R_0603_1608Metric_Pad0.98x0.95mm_HandSolder" (at 153.67 49.022 90)
       (effects (font (size 1.27 1.27)) hide)
     )
@@
       (effects (font (size 1.27 1.27)))
     )
-    (property "Footprint" "" (at 161.29 36.83 0)
+    (property "Footprint" "Diode_SMD:D_0201_0603Metric_Pad0.64x0.40mm_HandSolder" (at 161.29 36.83 0)
       (effects (font (size 1.27 1.27)) hide)
     )
@@
       (effects (font (size 1.27 1.27)) (justify left))
     )
-    (property "Footprint" "" (at 149.86 135.89 0)
-      (effects (font (size 1.27 1.27)) hide)
-    )
+    (property "Footprint" "MountingHole:MountingHole_2.2mm_M2_DIN965_Pad" (at 149.86 135.89 0)
+      (effects (font (size 1.27 1.27)) hide)
+    )

Commit message: Kikad Sch ok
Parts:
- added J5: Conn_02x04_Odd_Even, symbol Connector_Generic:Conn_02x04_Odd_Even
- C1, C2: footprint Capacitor_SMD:C_0805_2012Metric_Pad1.18x1.45mm_HandSolder -> (none)
- C3: value 1µF -> 1uF; footprint Capacitor_SMD:C_0805_2012Metric_Pad1.18x1.45mm_HandSolder -> (none)
- D1, D2: footprint Diode_SMD:D_0201_0603Metric_Pad0.64x0.40mm_HandSolder -> (none)
- H1, H2, H3, H4: footprint MountingHole:MountingHole_2.2mm_M2_DIN965_Pad -> (none)
- R1, R2, R3, R4, R5: footprint Resistor_SMD:R_0603_1608Metric_Pad0.98x0.95mm_HandSolder -> (none)
Connections:
- net +3.3V: now also J5.1 (Pin_1)
- net Debug_SWCLK: now also J5.2 (Pin_2)
- net Debug_SWDIO: now also J5.4 (Pin_4)
- net GND: now also C3.1, J5.8 (Pin_8); no longer C3.2
- net GPIO_Input: now also U1.1 (PB8); no longer U1.14 (PB1)
- net Interupteur: now also U1.14 (PB1); no longer U1.10 (PA4)
- net LED_Status_1: now also U1.2 (PF0); no longer U1.8 (PA2)
- net LED_Status_2: now also U1.3 (PF1); no longer U1.9 (PA3)
- net NRST: now reaches SW1.2, U1.4 (NRST)
- net NRST: now also C3.2, J5.6 (Pin_6); no longer C3.1
- new net USART2_RX: J5.3 (Pin_3), U1.9 (PA3)
- new net USART2_TX: J5.5 (Pin_5), U1.8 (PA2)
Other:
- note added: "CAN_Connector"
- note added: "SWD_Connector"
- note removed: "Connector"
- moved on the sheet: C1, C2, D1, D2, H1, H2, H3, H4, J1, J2, J3, R1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

Commit message: modif kicad indications
Parts:
- removed J5: Conn_02x04_Odd_Even, symbol Connector_Generic:Conn_02x04_Odd_Even
- added D3: LED, symbol Device:LED
- added J4: Conn_01x06_Pin, symbol Connector:Conn_01x06_Pin
- added J5: Conn_01x04_Pin, symbol Connector:Conn_01x04_Pin
- added J6: Conn_01x02_Pin, symbol Connector:Conn_01x02_Pin
- added R6: 1k, symbol Device:R
Connections:
- net +3.3V: now also D3.2 (A), J4.1 (Pin_1), J5.4 (Pin_4); no longer C2.1, U2.3 (VI)
- net Debug_SWCLK: now also J4.2 (Pin_2)
- net Debug_SWDIO: now also J4.4 (Pin_4)
- net GND: now also J4.3 (Pin_3), J5.3 (Pin_3), J6.2 (Pin_2), R6.2
- net NRST: now also J4.5 (Pin_5)
- net USART2_RX: now also J5.1 (Pin_1)
- net USART2_TX: now also J5.2 (Pin_2)
- net at SW2.1 (A): now also J6.1 (Pin_1)
- net Interupteur: no longer names the net of U1.14 (PB1)
- net Interupteur: no longer SW2.2 (B)
- new net: D3.1 (K), R6.1
- new net Alimentation: C2.1, SW2.2 (B), U2.3 (VI)
Other:
- note added: "Bluetooth connexion usart"
- note added: "LEDs"
- note added: "Power_Connector"
- note added: "Transciever CAN"
- note removed: "CAN"
- note removed: "LEDs + interrupteur"

Commit message: Datasheet regulateur
Parts:
- added C4: 100nF, symbol Device:C
- added R7: 120, symbol Device:R
- added SW3: SW_Push, symbol Switch:SW_Push
Connections:
- net +3.3VA is gone; now on net +3.3V: U1.5 (VDDA)
- net TIM2_CH1 is gone; now on net SD_card_detection: U1.6 (PA0)
- net +3.3V: now also C4.1
- net CAN_H: now also R7.1
- net CAN_L: now also R7.2
- net GND: now also C4.2, SW3.2
- net SD_CS: now reaches U1.10 (PA4)
- net SD_CS: now also J1.1 (CD/DAT3)
- net SD_card_detection: now reaches J1.10 (CARD_DETECT)
- net GPIO_Input renamed Test_PB
- net Test_PB: now also SW3.1
- net TIM2_CH2: no longer names the net of U1.7 (PA1)
- no-connect marks 8 -> 6
Other:
- note added: "Debug test"
- note removed: "LEDs"

Commit message: Kikad final
Parts:
- added C5: 10µF, symbol Device:C
- added D4: LED, symbol Device:LED
- added R8: 1k, symbol Device:R
- added U5: LM1117DT-5.0, Package_TO_SOT_SMD:TO-252-3_TabPin2, symbol Regulator_Linear:LM1117DT-5.0
- C4: value 100nF -> 10µF
- R7: value 120 -> R
Connections:
- net +3.3V: now also C5.1, D4.2 (A), U5.2 (VO); no longer C4.1
- net Alimentation: now also C4.1, U5.3 (VI)
- net GND: now also SW3.1, C5.2, R8.2, U5.1 (GND); no longer SW3.2
- net Test_PB: now also SW3.2; no longer SW3.1
- net SD_card_detection renamed SD_card_détection
- new net: D4.1 (K), R8.1
Other:
- note added: "LEDs"
- note added: "SD_Card"
- note removed: "Debug test"
- note removed: "SD_card"
- moved on the sheet: C1, C2, D3, H1, H2, H3, H4, J1, J4, J5, J6, R3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

Commit message: Schéma kicad avec empreinte
Parts:
- added C6: 100nF, Capacitor_SMD:C_0603_1608Metric_Pad1.08x0.95mm_HandSolder, symbol Device:C
- C1, C2, C3, C4, C5: footprint (none) -> Capacitor_SMD:C_0603_1608Metric_Pad1.08x0.95mm_HandSolder
- D1, D2, D3, D4: footprint (none) -> Diode_SMD:D_0603_1608Metric_Pad1.05x0.95mm_HandSolder
- H1, H2, H3, H4: footprint (none) -> MountingHole:MountingHole_3.2mm_M3_DIN965_Pad
- J1: footprint (none) -> Connector_Card:microSD_HC_Molex_104031-0811
- J2, J3: footprint (none) -> Connector:FanPinHeader_1x03_P2.54mm_Vertical
- J4: footprint (none) -> Connector_PinHeader_2.54mm:PinHeader_1x06_P2.54mm_Vertical
- J5: footprint (none) -> Connector:FanPinHeader_1x04_P2.54mm_Vertical
- J6: footprint (none) -> Connector_JST:JST_XH_B2B-XH-A_1x02_P2.50mm_Vertical
- R1, R2, R3, R4, R5, R6, R7, R8: footprint (none) -> Resistor_SMD:R_0603_1608Metric_Pad0.98x0.95mm_HandSolder
- SW1, SW2, SW3: footprint (none) -> Button_Switch_SMD:SW_SPST_EVQPE1
Connections:
- net +3.3V: now also C6.1
- net GND: now also C6.2

Commit message: re datalog
Parts:
- C1, C2, C3, C4, C5, C6: footprint Capacitor_SMD:C_0603_1608Metric_Pad1.08x0.95mm_HandSolder -> (none)
- D1, D2, D3, D4: footprint Diode_SMD:D_0603_1608Metric_Pad1.05x0.95mm_HandSolder -> (none)
- H1, H2, H3, H4: footprint MountingHole:MountingHole_3.2mm_M3_DIN965_Pad -> (none)
- J1: footprint Connector_Card:microSD_HC_Molex_104031-0811 -> (none)
- J2, J3: footprint Connector:FanPinHeader_1x03_P2.54mm_Vertical -> (none)
- J4: footprint Connector_PinHeader_2.54mm:PinHeader_1x06_P2.54mm_Vertical -> (none)
- J5: footprint Connector:FanPinHeader_1x04_P2.54mm_Vertical -> (none)
- J6: footprint Connector_JST:JST_XH_B2B-XH-A_1x02_P2.50mm_Vertical -> (none)
- R1, R2, R3, R4, R5, R6, R8: footprint Resistor_SMD:R_0603_1608Metric_Pad0.98x0.95mm_HandSolder -> (none)
- R7: value R -> 120; footprint Resistor_SMD:R_0603_1608Metric_Pad0.98x0.95mm_HandSolder -> (none)
- SW1, SW2, SW3: footprint Button_Switch_SMD:SW_SPST_EVQPE1 -> (none)
Other:
- moved on the sheet: R7, U3

Commit message: DATALOGGER avec empreinte
Parts:
- C1, C2, C3, C4, C5, C6: footprint (none) -> Capacitor_SMD:C_0603_1608Metric_Pad1.08x0.95mm_HandSolder
- D1, D2, D3, D4: footprint (none) -> Diode_SMD:D_0603_1608Metric_Pad1.05x0.95mm_HandSolder
- H1, H2, H3, H4: footprint (none) -> MountingHole:MountingHole_3.2mm_M3_DIN965_Pad
- J1: footprint (none) -> Connector_Card:microSD_HC_Molex_104031-0811
- J2, J3: footprint (none) -> Connector:FanPinHeader_1x03_P2.54mm_Vertical
- J4: footprint (none) -> Connector_PinHeader_2.54mm:PinHeader_1x06_P2.54mm_Vertical
- J5: footprint (none) -> Connector:FanPinHeader_1x04_P2.54mm_Vertical
- J6: footprint (none) -> Connector_JST:JST_XH_B2B-XH-A_1x02_P2.50mm_Vertical
- R1, R2, R3, R4, R5, R6, R7, R8: footprint (none) -> Resistor_SMD:R_0603_1608Metric_Pad0.98x0.95mm_HandSolder
- SW1, SW2, SW3: footprint (none) -> Button_Switch_SMD:SW_SPST_EVQPE1
Connections:
- net +3.3V: no longer C5.1, U3.3 (VDD), U5.2 (VO)
- new net 5V: C5.1, U3.3 (VDD), U5.2 (VO)
