File: Datalogger/Hardware/Datalogger.kicad_pcb (KiCad board)
At the start: 2 copper layers, 35 parts, among them J1 SD_Card, J2 Conn_01x03_Pin, J3 Conn_01x03_Pin, J4 Conn_01x06_Pin, J5 Conn_01x04_Pin, J6 Conn_01x02_Pin, SW1 SW_Push, SW2 SW_SPST, SW3 SW_Push, U1 STM32F042F6Px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

Commit message: Datalogger 19/02/2026 8h
Parts:
- J1: value SD_Card -> Micro_SD_Card; footprint Connector_Card:microSD_HC_Molex_104031-0811 -> Connector_Card:microSD_HC_Hirose_DM3AT-SF-PEJM5
- moved SW3 34.1 mm to (153.5, 64.5)
- moved U1 26.0 mm to (161.6, 72.2)
- moved J1 21.0 mm to (157.5, 50.0), turned to 180 degrees
- moved C6 20.4 mm to (167.1, 63.0)
- moved J6 15.5 mm to (190.0, 95.5)
- moved J3 9.81 mm to (169.9, 97.0)
- moved J4 9.02 mm to (186.5, 62.4)
- moved U5 8.86 mm to (176.9, 67.5)
- moved U2 8.35 mm to (176.8, 60.1)
Connections:
- J1 pad 1: SD_CS -> unconnected-(J1-DAT2-Pad1)
- J1 pad 10: SD_card_détection -> (no net)
- J1 pad 11: unconnected-(J1-WRITE_PROTECT-Pad11)_1 -> (no net)
- J1 pad 2: SD_SPI1_MOSI -> SD_CS
- J1 pad 3: GND -> SD_SPI1_MOSI
- J1 pad 9: unconnected-(J1-DAT2-Pad9) -> GND
- U1 pad 6: SD_card_détection -> unconnected-(U1-PA0-Pad6)
