File: Odometre/Hardware/Odometre_Schematic/Odometre_Schematic-backups/Odometre_Schematic-2026-02-18_171104/Odometre_Schematic.kicad_pcb (KiCad board)
At the start: 2 copper layers, 35 parts, among them IC1 STM32C092FCP6, J1 Conn_01x03_Pin, J2 Conn_01x03_Pin, J3 Conn_Alim, J4 Conn_Laser1, J5 Conn_Laser2, J6 Conn_01x06_Pin, J7 Conn_01x06_Pin, SW1 Reset_Botton, SW2 Debug_Botton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

Commit message: schematic vf
Parts:
- J4, J5: footprint Connector_PinSocket_2.54mm:PinSocket_1x02_P2.54mm_Vertical -> Connector:FanPinHeader_1x03_P2.54mm_Vertical
- J6, J7: footprint Connector_PinHeader_2.54mm:PinHeader_1x03_P2.54mm_Vertical -> Connector_PinHeader_2.54mm:PinHeader_1x06_P2.54mm_Vertical
- moved H3 71.1 mm to (180.0, 150.0)
- moved D4 62.0 mm to (118.0, 63.5), turned to 180 degrees
- moved H2 61.1 mm to (180.0, 50.0)
- moved J3 60.9 mm to (119.0, 69.0)
- moved U3 58.5 mm to (109.0, 70.3), turned to 90 degrees
- moved H4 57.5 mm to (100.0, 150.5)
- moved R5 57.3 mm to (121.9, 63.5)
- moved U2 50.2 mm to (109.2, 86.5), turned to 180 degrees
- moved H1 46.2 mm to (100.0, 50.0)
- moved R4 40.2 mm to (126.5, 93.0), turned to 180 degrees
- moved C8 31.7 mm to (119.8, 76.0)
- moved D3 29.8 mm to (130.6, 93.0)
- moved C9 28.6 mm to (120.0, 83.0)
- moved R3 28.3 mm to (176.5, 68.1)
- moved D1 28.3 mm to (164.4, 79.5)
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Connections:
- C1 pad 1: ALIM_Trans -> Alim
- C8 pad 1: ALIM_Trans -> Alim
- J3 pad 1: ALIM_Trans -> Alim
- U2 pad 3: ALIM_Trans -> Alim
- U3 pad 3: ALIM_Trans -> Alim
Routing:
- added copper zone on B.Cu, net (none)
- added copper zone on F.Cu, net (none)
Other:
- board outline added: 90 x 110.5 mm

Commit message: schematic et pcb
Parts:
- moved J7 73.3 mm to (138.0, 121.5), turned to -90 degrees
- moved J5 54.8 mm to (129.0, 112.5), turned to 180 degrees
- moved J4 47.1 mm to (133.9, 112.0)
- moved R1 46.9 mm to (151.9, 103.0)
- moved U1 44.2 mm to (151.5, 93.4)
- moved J6 43.8 mm to (133.8, 87.0), turned to 90 degrees
- moved J1 35.4 mm to (163.9, 88.4)
- moved J2 35.4 mm to (168.5, 88.4)
- moved C9 34.5 mm to (146.1, 60.5)
- moved R3 31.0 mm to (157.9, 92.9), turned to -90 degrees
- moved C8 28.7 mm to (146.0, 64.0)
- moved C1 28.7 mm to (146.0, 67.5)
- moved D1 28.4 mm to (148.4, 103.0), turned to 180 degrees
- moved U2 27.5 mm to (135.6, 78.5)
- moved R5 27.5 mm to (148.3, 55.5)
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Connections:
- J6 pad 3: GND -> unconnected-(J6-Pin_3-Pad3)
- J6 pad 6: unconnected-(J6-Pin_6-Pad6) -> GND
- J7 pad 4: TIM2_CH2 -> VDD/VDDA
- J7 pad 5: VDD/VDDA -> TIM2_CH2
