File: Odometre/Hardware/Odometre_Schematic/Odometre_Schematic-backups/Odometre_Schematic-2026-02-18_171104/_autosave-Odometre_Schematic.kicad_sch (KiCad schematic)
At the start: 35 parts, among them IC1 STM32C092FCP6, J1 Conn_01x03_Pin, J2 Conn_01x03_Pin, J3 Conn_Alim, J4 Conn_Laser1, J5 Conn_Laser2, J6 Conn_01x06_Pin, J7 Conn_01x06_Pin, SW1 Reset_Botton, SW2 Debug_Botton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

Commit message: schematic et pcb
Connections:
- net +3.3V: now also J7.4 (Pin_4); no longer J7.5 (Pin_5)
- net GND: now also J6.6 (Pin_6); no longer J6.3 (Pin_3)
- net TIM2_CH2: now also J7.5 (Pin_5); no longer J7.4 (Pin_4)
Changed lines of the file:
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@@
 	)
 	(rectangle
-		(start 69.85 165.1)
-		(end 106.68 191.77)
+		(start 68.58 165.1)
+		(end 105.41 191.77)
 		(stroke
 			(width 0)
@@
 	)
 	(no_connect
-		(at 44.45 144.78)
-	)
-	(no_connect
 		(at 35.56 55.88)
 	)
@@
 		(at 35.56 38.1)
 	)
+	(no_connect
+		(at 44.45 137.16)
+	)
 	(wire
 		(pts
@@
 	(wire
 		(pts
+			(xy 88.9 180.34) (xy 92.71 180.34)
+		)
+		(stroke
+			(width 0)
+			(type default)
+		)
+	)
+	(wire
+		(pts
 			(xy 252.73 45.72) (xy 252.73 54.61)
 		)
@@
 	(wire
 		(pts
+			(xy 88.9 177.8) (xy 87.63 177.8)
+		)
+		(stroke
+			(width 0)
+			(type default)
+		)
+	)
+	(wire
+		(pts
 			(xy 215.9 87.63) (xy 217.17 87.63)
 		)
@@
 		)
 	)
-	(global_label "TIM2_CH1"
+	(global_label "VDD{slash}VDDA"
 		(shape input)
-		(at 88.9 180.34 0)
+		(at 189.23 60.96 90)
 		(fields_autoplaced yes)
 		(effects
@@
 		)
 		(property "Intersheetrefs" "${INTERSHEET_REFS}"
-			(at 100.8167 180.34 0)
+			(at 189.23 48.3779 90)
 			(effects
 				(font
@@
 		)
 	)
-	(global_label "VDD{slash}VDDA"
+	(global_label "FDCAN1_RX"
 		(shape input)
-		(at 189.23 60.96 90)
+		(at 88.9 48.26 0)
 		(fields_autoplaced yes)
 		(effects
@@
 		)
 		(property "Intersheetrefs" "${INTERSHEET_REFS}"
-			(at 189.23 48.3779 90)
+			(at 102.5101 48.26 0)
 			(effects
 				(font
@@
 		)
 	)
-	(global_label "FDCAN1_RX"
+	(global_label "CANH"
 		(shape input)
-		(at 88.9 48.26 0)
+		(at 232.41 39.37 90)
 		(fields_autoplaced yes)
 		(effects
@@
 		)
 		(property "Intersheetrefs" "${INTERSHEET_REFS}"
-			(at 102.5101 48.26 0)
+			(at 232.41 31.4446 90)
 			(effects
 				(font
@@
 		)
 	)
-	(global_label "CANH"
+	(global_label "Green_LED"
 		(shape input)
-		(at 232.41 39.37 90)
+		(at 88.9 45.72 0)
 		(fields_autoplaced yes)
 		(effects
@@
 		)
 		(property "Intersheetrefs" "${INTERSHEET_REFS}"
-			(at 232.41 31.4446 90)
+			(at 101.6029 45.72 0)
 			(effects
 				(font
@@
 		)
 	)
-	(global_label "Green_LED"
+	(global_label "TIM2_CH2"
 		(shape input)
-		(at 88.9 45.72 0)
+		(at 88.9 185.42 0)
 		(fields_autoplaced yes)
 		(effects
@@
 		)
 		(property "Intersheetrefs" "${INTERSHEET_REFS}"
-			(at 101.6029 45.72 0)
+			(at 100.8961 185.42 0)
 			(effects
 				(font
@@
 		)
 	)
+	(global_label "TIM2_CH1"
+		(shape input)
+		(at 92.71 180.34 0)
+		(fields_autoplaced yes)
+		(effects
+			(font
+				(size 1.27 1.27)
+			)
+			(justify left)
+		)
+		(property "Intersheetrefs" "${INTERSHEET_REFS}"
+			(at 104.6267 180.34 0)
+			(effects
+				(font
+					(size 1.27 1.27)
+				)
+				(justify left)
+				(hide yes)
+			)
+		)
+	)
 	(global_label "CANH"
 		(shape input)
@@
 		)
 	)
-	(global_label "TIM2_CH2"
-		(shape input)
-		(at 88.9 182.88 0)
-		(fields_autoplaced yes)
-		(effects
-			(font
-				(size 1.27 1.27)
-			)
-			(justify left)
-		)
-		(property "Intersheetrefs" "${INTERSHEET_REFS}"
-			(at 100.8167 182.88 0)
-			(effects
-				(font
-					(size 1.27 1.27)
-				)
-				(justify left)
-				(hide yes)
-			)
-		)
-	)
 	(global_label "NRST"
 		(shape input)
@@
 	)
 	(symbol
-		(lib_id "power:+3.3V")
-		(at 88.9 185.42 270)
+		(lib_id "power:GND")
+		(at 166.37 55.88 90)
 		(unit 1)
 		(exclude_from_sim no)
@@
 		(dnp no)
 		(fields_autoplaced yes)
-		(property "Reference" "#PWR025"
-			(at 85.09 185.42 0)
+		(property "Reference" "#PWR011"
+			(at 172.72 55.88 0)
 			(effects
 				(font
@@
 			)
 		)
-		(property "Value" "+3.3V"
-			(at 92.71 186.055 90)
+		(property "Value" "GND"
+			(at 170.18 56.515 90)
 			(effects
 				(font
 					(size 1.27 1.27)
 				)
-				(justify left)
+				(justify right)
 			)
 		)
 		(property "Footprint" ""
-			(at 88.9 185.42 0)
+			(at 166.37 55.88 0)
 			(effects
 				(font
@@
 		)
 		(property "Datasheet" ""
-			(at 88.9 185.42 0)
+			(at 166.37 55.88 0)
 			(effects
 				(font
@@
 		)
 		(property "Description" ""
-			(at 88.9 185.42 0)
+			(at 166.37 55.88 0)
 			(effects
 				(font
@@
 			(project "Odometre_Schematic"
 				(path "/3741a7b9-879e-49a1-88bd-82d63456a983"
-					(reference "#PWR025")
+					(reference "#PWR011")
 					(unit 1)
 				)
@@
 	)
 	(symbol
-		(lib_id "power:GND")
-		(at 166.37 55.88 90)
+		(lib_id "power:+3.3V")
+		(at 88.9 182.88 270)
 		(unit 1)
 		(exclude_from_sim no)
@@
 		(on_board yes)
 		(dnp no)
-		(fields_autoplaced yes)
-		(property "Reference" "#PWR011"
-			(at 172.72 55.88 0)
+		(property "Reference" "#PWR025"
+			(at 85.09 182.88 0)
 			(effects
 				(font
@@
 			)
 		)
-		(property "Value" "GND"
-			(at 170.18 56.515 90)
+		(property "Value" "+3.3V"
+			(at 92.71 183.515 90)
 			(effects
 				(font
 					(size 1.27 1.27)
 				)
-				(justify right)
+				(justify left)
 			)
 		)
 		(property "Footprint" ""
-			(at 166.37 55.88 0)
+			(at 88.9 182.88 0)
 			(effects
 				(font
@@
 		)
 		(property "Datasheet" ""
-			(at 166.37 55.88 0)
+			(at 88.9 182.88 0)
 			(effects
 				(font
@@
 		)
 		(property "Description" ""
-			(at 166.37 55.88 0)
+			(at 88.9 182.88 0)
 			(effects
 				(font
@@
 			(project "Odometre_Schematic"
 				(path "/3741a7b9-879e-49a1-88bd-82d63456a983"
-					(reference "#PWR011")
+					(reference "#PWR025")
 					(unit 1)
 				)
@@
 	(symbol
 		(lib_id "power:GND")
-		(at 44.45 137.16 90)
+		(at 44.45 144.78 90)
 		(unit 1)
 		(exclude_from_sim no)
@@
 		(fields_autoplaced yes)
 		(property "Reference" "#PWR013"
-			(at 50.8 137.16 0)
+			(at 50.8 144.78 0)
 			(effects
 				(font
@@
 		)
 		(property "Value" "GND"
-			(at 48.26 137.795 90)
+			(at 48.26 145.415 90)
 			(effects
 				(font
@@
 		)
 		(property "Footprint" ""
-			(at 44.45 137.16 0)
+			(at 44.45 144.78 0)
 			(effects
 				(font
@@
 		)
 		(property "Datasheet" ""
-			(at 44.45 137.16 0)
+			(at 44.45 144.78 0)
 			(effects
 				(font
@@
 		)
 		(property "Description" ""
-			(at 44.45 137.16 0)
+			(at 44.45 144.78 0)
 			(effects
 				(font
@@
 	(symbol
 		(lib_id "power:GND")
-		(at 88.9 177.8 90)
+		(at 87.63 177.8 90)
 		(unit 1)
 		(exclude_from_sim no)
@@
 		(fields_autoplaced yes)
 		(property "Reference" "#PWR023"
-			(at 95.25 177.8 0)
+			(at 93.98 177.8 0)
 			(effects
 				(font
@@
 		)
 		(property "Value" "GND"
-			(at 92.71 178.435 90)
+			(at 91.44 178.435 90)
 			(effects
 				(font
@@
 		)
 		(property "Footprint" ""
-			(at 88.9 177.8 0)
+			(at 87.63 177.8 0)
 			(effects
 				(font
@@
 		)
 		(property "Datasheet" ""
-			(at 88.9 177.8 0)
+			(at 87.63 177.8 0)
 			(effects
 				(font
@@
 		)
 		(property "Description" ""
-			(at 88.9 177.8 0)
+			(at 87.63 177.8 0)
 			(effects
 				(font
