File: Datalogger/Hardware/Dataloggerdusoir/datalogger2/datalogger2.kicad_sch (KiCad schematic)
At the start: 35 parts, among them J1 Micro_SD_Card, J2 Conn_01x03_Pin, J3 Conn_01x03_Pin, J4 Conn_01x06_Pin, J5 Conn_01x04_Pin, J6 Conn_01x02_Pin, SW1 SW_Push, SW2 SW_SPST, SW3 SW_Push, U1 STM32F042F6Px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

Commit message: Datalogger 19/02/2026 13:33
Parts:
- added C7, C8: 100nF, Capacitor_SMD:C_0805_2012Metric_Pad1.18x1.45mm_HandSolder, symbol Device:C
- C1, C2, C3, C4, C5, C6: footprint Capacitor_SMD:C_0603_1608Metric_Pad1.08x0.95mm_HandSolder -> Capacitor_SMD:C_0805_2012Metric_Pad1.18x1.45mm_HandSolder
- R1, R2, R3, R4, R5, R6, R7, R8: footprint Resistor_SMD:R_0603_1608Metric_Pad0.98x0.95mm_HandSolder -> Resistor_SMD:R_0805_2012Metric_Pad1.20x1.40mm_HandSolder
- SW1, SW3: footprint Button_Switch_THT:SW_PUSH_6mm -> Button_Switch_SMD:SW_Tactile_SPST_NO_Straight_CK_PTS636Sx25SMTRLFS
- SW2: footprint Button_Switch_THT:SW_PUSH_6mm -> Button_Switch_THT:SW_SPST_Omron_B3F-40xx
Connections:
- net +3.3V: now also C7.1, C8.1; no longer C6.1, D4.2 (A)
- net 5V: now also C6.1, D4.2 (A)
- net GND: now also C7.2, C8.2
