File: Datalogger/Hardware/Dataloggerdusoir/datalogger2/datalogger2.kicad_pcb (KiCad board)
At the start: 2 copper layers, 60 x 65 mm, 35 parts, among them J1 Micro_SD_Card, J2 Conn_01x03_Pin, J3 Conn_01x03_Pin, J4 Conn_01x06_Pin, J5 Conn_01x04_Pin, J6 Conn_01x02_Pin, SW1 SW_Push, SW2 SW_SPST, SW3 SW_Push, U1 STM32F042F6Px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

Commit message: Datalogger 19/02/2026 13:33
Parts:
- added C7: 100nF, Capacitor_SMD:C_0805_2012Metric_Pad1.18x1.45mm_HandSolder, F.Cu at (164.3, 57.0)
- added C8: 100nF, Capacitor_SMD:C_0805_2012Metric_Pad1.18x1.45mm_HandSolder, F.Cu at (150.9, 56.4)
- C1, C2, C3, C4, C5, C6: footprint Capacitor_SMD:C_0603_1608Metric_Pad1.08x0.95mm_HandSolder -> Capacitor_SMD:C_0805_2012Metric_Pad1.18x1.45mm_HandSolder
- R1, R2, R3, R4, R5, R6, R7, R8: footprint Resistor_SMD:R_0603_1608Metric_Pad0.98x0.95mm_HandSolder -> Resistor_SMD:R_0805_2012Metric_Pad1.20x1.40mm_HandSolder
- SW1, SW3: footprint Button_Switch_THT:SW_PUSH_6mm -> Button_Switch_SMD:SW_Tactile_SPST_NO_Straight_CK_PTS636Sx25SMTRLFS
- SW2: footprint Button_Switch_THT:SW_PUSH_6mm -> Button_Switch_THT:SW_SPST_Omron_B3F-40xx
- moved SW1 43.9 mm to (175.6, 35.6)
- moved SW3 36.8 mm to (140.6, 55.2)
- moved D3 31.5 mm to (175.8, 77.2)
- moved C6 30.7 mm to (166.6, 64.8), turned to 90 degrees
- moved C4 24.8 mm to (166.3, 43.3)
- moved C5 23.7 mm to (162.5, 43.3), turned to 180 degrees
- moved R3 22.4 mm to (159.6, 74.4), turned to 90 degrees
- moved R4 16.9 mm to (159.6, 70.4), turned to 90 degrees
- moved D4 16.6 mm to (175.8, 80.0)
- moved J4 15.7 mm to (176.4, 89.2), turned to -90 degrees
- moved SW2 15.5 mm to (172.0, 46.3)
- moved R8 15.5 mm to (175.8, 82.5)
- moved R2 13.2 mm to (155.1, 47.3)
- moved R6 13.1 mm to (175.7, 74.2)
- moved R7 13.0 mm to (178.0, 64.7), turned to -90 degrees
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Connections:
- C6 pad 1: +3.3V -> 5V
- D4 pad 2: +3.3V -> 5V
Routing:
- net +3.3V: track 0.00 -> 142.0 mm, vias 0 -> 3
- net NRST: track 0.00 -> 94.6 mm, vias 0 -> 5
- net Alimentation: track 0.00 -> 88.1 mm
- net 5V: track 0.00 -> 59.6 mm, vias 0 -> 4
- net Debug_SWCLK: track 0.00 -> 43.0 mm, vias 0 -> 2
- net Debug_SWDIO: track 0.00 -> 42.0 mm, vias 0 -> 2
- net CAN_H: track 0.00 -> 30.2 mm
- net SD_SPI1_SCK: track 0.00 -> 29.2 mm, vias 0 -> 2
- net SD_SPI1_MOSI: track 0.00 -> 28.8 mm
- net Net-(J6-Pin_1): track 0.00 -> 27.3 mm
- net CAN_RX: track 0.00 -> 26.2 mm
- net CAN_L: track 0.00 -> 24.6 mm
- net SD_CS: track 0.00 -> 22.8 mm, vias 0 -> 2
- net USART2_TX: track 0.00 -> 22.1 mm
- net USART2_RX: track 0.00 -> 20.9 mm, vias 0 -> 2
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Other:
- outline, holes or cut-outs redrawn

Commit message: Datalogger Final
Routing:
- net GND: track 6.96 -> 185.1 mm, vias 0 -> 8
- net SD_SPI1_MISO: track 16.9 -> 26.4 mm

Commit message: Modification PCB pour impression
Other:
- board text added: "Joseph GERVAIS, ENSEA CAN Datalogger"
Changed lines of the file:
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@@
 			(outputformat 1)
 			(mirror no)
-			(drillshape 1)
+			(drillshape 0)
 			(scaleselection 1)
-			(outputdirectory "")
+			(outputdirectory "fichier_gerber_fabrication/")
 		)
 	)
@@
 			(at 2.5 -3.4 90)
 			(layer "F.SilkS")
+			(hide yes)
 			(effects
 				(font
@@
 			(at 0 -1.65 0)
 			(layer "F.SilkS")
+			(hide yes)
 			(effects
 				(font
@@
 			(at 0 1.65 0)
 			(layer "F.Fab")
+			(hide yes)
 			(effects
 				(font
@@
 			(at 0 -1.43 0)
 			(layer "F.SilkS")
+			(hide yes)
 			(effects
 				(font
@@
 			(at 0 -1.43 0)
 			(layer "F.SilkS")
+			(hide yes)
 			(effects
 				(font
@@
 			(at -0.25 -4.18 0)
 			(layer "F.SilkS")
+			(hide yes)
 			(effects
 				(font
@@
 		(layer "Edge.Cuts")
 	)
+	(gr_text "Joseph GERVAIS, ENSEA\nCAN Datalogger"
+		(at 166 86 90)
+		(layer "F.SilkS")
+		(effects
+			(font
+				(size 1 1)
+				(thickness 0.15)
+			)
+			(justify left bottom)
+		)
+	)
 	(segment
