File: gestionnaire de batterie/PCB/Odometre_Schematic.kicad_pcb (KiCad board)
At the start: 2 copper layers, 83.2 x 61.6 mm, 40 parts, among them IC1 STM32C092FCP6, J1 Conn_01x03_Pin, J2 Conn_01x03_Pin, J3 Conn_Alim, J6 Conn_SWD, U1 MCP2562-E-SN, U2 LM1117DT-3.3, U3 LM1117DT-5.0, U4 LA55-P

Commit message: Création des fichiers de fabrication
Other:
- board text added: "Formula Student ENSEA Arthur VENTURA BMS"
Changed lines of the file:
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@@
 			(outputformat 1)
 			(mirror no)
-			(drillshape 1)
+			(drillshape 0)
 			(scaleselection 1)
-			(outputdirectory "")
+			(outputdirectory "Fabrication/")
 		)
 	)
@@
 		(layer "Edge.Cuts")
 	)
+	(gr_text "Formula Student ENSEA\nArthur VENTURA\nBMS"
+		(at 165.5 132.5 90)
+		(layer "F.SilkS")
+		(effects
+			(font
+				(size 1.5 1.5)
+				(thickness 0.2)
+			)
+			(justify left bottom)
+		)
+	)
 	(segment
